Commit message: Tele Operation for Robot Added

File: urdf/model.gazebo.xacro (robot description, xacro)
@@ -97,5 +97,5 @@
       <leftJoint>front_left_wheel</leftJoint>
       <rightJoint>front_right_wheel</rightJoint>
-      <wheelSeparation>0.160</wheelSeparation>
+      <wheelSeparation>0.160</wheelSeparation>				<!--TODO-->
       <wheelDiameter>0.066</wheelDiameter>
       <wheelAcceleration>1</wheelAcceleration>

File: urdf/model.urdf.xacro (robot description, xacro)
@@ -9,4 +9,5 @@
 	<xacro:property name="base_to_wheel_y" value="0.075" />
 	<xacro:property name="base_to_wheel_z" value="-0.01" />
+	<xacro:property name="base_to_lds_yx" value="0.0" />
 	<xacro:property name="base_to_lds_y" value="0.1" />
 	<xacro:property name="base_to_lds_z" value="0.13" />

Commit message: Added support for Lidar Sensor

File: urdf/model.gazebo.xacro (robot description, xacro)
@@ -83,5 +83,5 @@
   <!-- Gazebo plugin for Driving Base -->
   <gazebo>
-    <plugin name="mcubot_burger_controller" filename="libgazebo_ros_diff_drive.so">
+    <plugin name="mcubot_base_controller" filename="libgazebo_ros_diff_drive.so">
       <commandTopic>cmd_vel</commandTopic>
       <odometryTopic>odom</odometryTopic>
@@ -104,4 +104,37 @@
     </plugin>
   </gazebo>
+  <!-- Gazebo plugin for Lidar Sensor -->
+  <gazebo reference="base_scan">
+    <material>Gazebo/FlatBlack</material>
+    <sensor type="ray" name="lds_lfcd_sensor">
+      <pose>0 0 0 0 0 0</pose>
+      <visualize>$(arg laser_visual)</visualize>
+      <update_rate>5</update_rate>
+      <ray>
+        <scan>
+          <horizontal>
+            <samples>360</samples>
+            <resolution>1</resolution>
+            <min_angle>0.0</min_angle>
+            <max_angle>6.28319</max_angle>
+          </horizontal>
+        </scan>
+        <range>
+          <min>0.120</min>
+          <max>3.5</max>
+          <resolution>0.015</resolution>
+        </range>
+        <noise>
+          <type>gaussian</type>
+          <mean>0.0</mean>
+          <stddev>0.01</stddev>
+        </noise>
+      </ray>
+      <plugin name="gazebo_ros_lds_lfcd_controller" filename="libgazebo_ros_laser.so">
+        <topicName>scan</topicName>
+        <frameName>base_scan</frameName>
+      </plugin>
+    </sensor>
+  </gazebo>
   <!-- Gazebo plugin for ROS Control -->
   <gazebo>
