Commit message: FIXED robot_state_publisher & KDL error

File: urdf/model.urdf.xacro (robot description, xacro)
@@ -12,4 +12,10 @@
 	<xacro:property name="base_to_lds_y" value="0.1" />
 	<xacro:property name="base_to_lds_z" value="0.13" />
+  <!-- DUMMY LINK TO AVOID KDL ERROR -->
+  <link name="dummy"/>
+  <joint name="dummy_joint" type="fixed">
+    <parent link="dummy"/>
+    <child link="base_link"/>
+  </joint>
   <!-- Base Link -->
   <link name="base_link">

Commit message: added navigation, updated deprecations, fixed errors/warnings

File: urdf/model.urdf.xacro (robot description, xacro)
@@ -9,13 +9,7 @@
 	<xacro:property name="base_to_wheel_y" value="0.075" />
 	<xacro:property name="base_to_wheel_z" value="-0.01" />
-	<xacro:property name="base_to_lds_yx" value="0.0" />
+	<xacro:property name="base_to_lds_x" value="0.0" />
 	<xacro:property name="base_to_lds_y" value="0.1" />
 	<xacro:property name="base_to_lds_z" value="0.13" />
-  <!-- DUMMY LINK TO AVOID KDL ERROR -->
-  <link name="dummy"/>
-  <joint name="dummy_joint" type="fixed">
-    <parent link="dummy"/>
-    <child link="base_link"/>
-  </joint>
   <!-- Base Link -->
   <link name="base_link">
@@ -28,9 +22,10 @@
     </visual>
     <collision>
-      <origin rpy="0 0 0" xyz="${base_link_x} ${base_link_y} ${base_link_z+0.045}"/>
+      <origin rpy="0 0 0" xyz="${base_link_x} ${base_link_y} ${base_link_z+0.040}"/>
       <geometry>
         <box size="0.25 0.32 0.14"/>
       </geometry>
     </collision>
+    <!--
     <inertial>
       <mass value="1" />
@@ -40,7 +35,8 @@
                izz="0.000025" />
     </inertial>
+    -->
   </link>
-  <!--Front Left Wheel-->
-  <link name="front_left_wheel">
+  <!--Front RIGHT Wheel-->
+  <link name="front_right_wheel">
 		<visual>
       <origin rpy="0 0 0" xyz="0 0 0"/>
@@ -51,5 +47,34 @@
     </visual>
     <collision>
-      <origin xyz="0.01 0 0" rpy="0 1.57 0"/>
+      <origin xyz="0.01 0 0" rpy="0 1.5708 0"/>
+      <geometry>
+        <cylinder length="0.015" radius="0.046"/>
+      </geometry>
+    </collision>
+    <inertial>
+      <mass value="0.1" />
+      <origin xyz="0 0 0" />
+      <inertia ixx="0.001" ixy="0.0" ixz="0.0"
+               iyy="0.001" iyz="0.0"
+               izz="0.001" />
+    </inertial>
+  </link>
+  <joint name="base_to_front_right_wheel" type="continuous">
+  	<origin rpy="0 0 0" xyz="${base_to_wheel_x} ${base_to_wheel_y} ${base_to_wheel_z}"/>
+  	<axis xyz="-1 0 0"/>
+    <parent link="base_link"/>
+    <child link="front_right_wheel"/>
+  </joint>
+  <!--Front LEFT Wheel-->
+  <link name="front_left_wheel">
+		<visual>
+      <origin rpy="0 0 3.1415" xyz="0 0 0"/>
+      <material name="white"/>
+      <geometry>
+        <mesh filename="package://mcubot/meshes/wheel.stl" scale="1 1 1"/>
+      </geometry>
+    </visual>
+    <collision>
+      <origin xyz="-0.01 0 0" rpy="0 1.5708 0"/>
       <geometry>
         <cylinder length="0.015" radius="0.046"/>
@@ -65,13 +90,13 @@
   </link>
   <joint name="base_to_front_left_wheel" type="continuous">
-  	<origin rpy="0 0 0" xyz="${base_to_wheel_x} ${base_to_wheel_y} ${base_to_wheel_z}"/>
-  	<axis xyz="1 0 0"/>
+  	<origin rpy="0 0 0" xyz="-${base_to_wheel_x} ${base_to_wheel_y} ${base_to_wheel_z}"/>
+  	<axis xyz="-1 0 0"/>
     <parent link="base_link"/>
     <child link="front_left_wheel"/>
   </joint>
-  <!--Front Right Wheel-->
-  <link name="front_right_wheel">
+  <!--Back RIGHT Wheel-->
+  <link name="back_right_wheel">
 		<visual>
-      <origin rpy="0 0 3.1415" xyz="0 0 0"/>
+      <origin rpy="0 0 0" xyz="0 0 0"/>
       <material name="white"/>
       <geometry>
@@ -80,5 +105,5 @@
     </visual>
     <collision>
-      <origin xyz="-0.01 0 0" rpy="0 1.57 0"/>
+      <origin xyz="0.01 0 0" rpy="0 1.5708 0"/>
       <geometry>
         <cylinder length="0.015" radius="0.046"/>
@@ -93,14 +118,14 @@
     </inertial>
   </link>
-  <joint name="base_to_front_right_wheel" type="continuous">
-  	<origin rpy="0 0 0" xyz="-${base_to_wheel_x} ${base_to_wheel_y} ${base_to_wheel_z}"/>
-  	<axis xyz="1 0 0"/>
+  <joint name="base_to_back_right_wheel" type="continuous">
+  	<origin rpy="0 0 0" xyz="${base_to_wheel_x} -${base_to_wheel_y} ${base_to_wheel_z}"/>
+  	<axis xyz="-1 0 0"/>
     <parent link="base_link"/>
-    <child link="front_right_wheel"/>
+    <child link="back_right_wheel"/>
   </joint>
-  <!--Back Left Wheel-->
+  <!--Back LEFT Wheel-->
   <link name="back_left_wheel">
 		<visual>
-      <origin rpy="0 0 0" xyz="0 0 0"/>
+      <origin rpy="0 0 3.1415" xyz="0 0 0"/>
       <material name="white"/>
       <geometry>
@@ -109,5 +134,5 @@
     </visual>
     <collision>
-      <origin xyz="0.01 0 0" rpy="0 1.57 0"/>
+      <origin xyz="-0.01 0 0" rpy="0 1.5708 0"/>
       <geometry>
         <cylinder length="0.015" radius="0.046"/>
@@ -123,42 +148,13 @@
   </link>
   <joint name="base_to_back_left_wheel" type="continuous">
-  	<origin rpy="0 0 0" xyz="${base_to_wheel_x} -${base_to_wheel_y} ${base_to_wheel_z}"/>
-  	<axis xyz="1 0 0"/>
+  	<origin rpy="0 0 0" xyz="-${base_to_wheel_x} -${base_to_wheel_y} ${base_to_wheel_z}"/>
+  	<axis xyz="-1 0 0"/>
     <parent link="base_link"/>
     <child link="back_left_wheel"/>
-  </joint>
-  <!--Back Right Wheel-->
-  <link name="back_right_wheel">
-		<visual>
-      <origin rpy="0 0 3.1415" xyz="0 0 0"/>
-      <material name="white"/>
-      <geometry>
-        <mesh filename="package://mcubot/meshes/wheel.stl" scale="1 1 1"/>
-      </geometry>
-    </visual>
-    <collision>
-      <origin xyz="-0.01 0 0" rpy="0 1.57 0"/>
-      <geometry>
-        <cylinder length="0.015" radius="0.046"/>
-      </geometry>
-    </collision>
-    <inertial>
-      <mass value="0.1" />
-      <origin xyz="0 0 0" />
-      <inertia ixx="0.001" ixy="0.0" ixz="0.0"
-               iyy="0.001" iyz="0.0"
-               izz="0.001" />
-    </inertial>
-  </link>
-  <joint name="base_to_back_right_wheel" type="continuous">
-  	<origin rpy="0 0 0" xyz="-${base_to_wheel_x} -${base_to_wheel_y} ${base_to_wheel_z}"/>
-  	<axis xyz="1 0 0"/>
-    <parent link="base_link"/>
-    <child link="back_right_wheel"/>
   </joint>
 	<!--Lidar Sensor-->
   <link name="base_scan">
     <visual>
-      <origin xyz="0 0 0.0" rpy="0 0 1.57"/>
+      <origin xyz="0 0 0.0" rpy="0 0 1.5708"/>
       <material name="black"/>
       <geometry>
@@ -168,5 +164,5 @@
     </visual>
     <collision>
-      <origin xyz="0 0 0" rpy="0 0 1.57"/>
+      <origin xyz="0 0 0" rpy="0 0 1.5708"/>
       <geometry>
         <cylinder length="0.0315" radius="0.055"/>
@@ -184,5 +180,5 @@
     <parent link="base_link"/>
     <child link="base_scan"/>
-    <origin xyz="0 ${base_to_lds_y} ${base_to_lds_z}" rpy="0 0 0"/>
+    <origin xyz="${base_to_lds_x} ${base_to_lds_y} ${base_to_lds_z}" rpy="0 0 0"/>
   </joint>
 </robot>
